File: Hardware/Electronics/CAD/MotorController.kicad_pcb (KiCad board)
At the start: 2 copper layers, 42.3 x 42.3 mm, 14 parts, among them J1 MPE 094-1-006, J2 CONN_01X03, J3 Screw_Terminal_1x02, J5 CONN_01X04, SW2 SW_DPST_x2, U1 LD1117S33CTR, U2 MAX471, U3 TMC2130, U4 ESP-12E, U5 HiLink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

Commit message: revision1.0.0 for electrical hardware
Parts:
- added R1: RND 0805 1 10K, Resistors_SMD:R_0805, F.Cu at (201.9, 41.5)
- added R2: RND 0805 1 10K, Resistors_SMD:R_0805, F.Cu at (205.3, 41.5)
- C1, C2, U1, U3, U4: moved to B.Cu
- J1: footprint Socket_Strips:Socket_Strip_Angled_1x06_Pitch2.54mm -> Pin_Headers:Pin_Header_Straight_1x06_Pitch2.54mm_SMD_Pin1Right
- J2: footprint Pin_Headers:Pin_Header_Angled_1x03_Pitch2.54mm -> Pin_Headers:Pin_Header_Straight_1x03_Pitch2.54mm_SMD_Pin1Right
- J3: footprint WAGO:WAGO_2pin -> Terminal:SolderTerminal; moved to B.Cu
- J5: footprint Pin_Headers:Pin_Header_Angled_1x04_Pitch2.54mm -> Terminal:Pin_Header_SMD_Angled_2.54mm
- U5: footprint HiLink:HiLink -> HiLink:HLK-PM01
- moved R5 54.5 mm to (201.2, 71.4), turned to 90 degrees
- moved SW2 39.1 mm to (205.2, 74.1), turned to 270 degrees
- moved J2 35.2 mm to (190.2, 71.7), turned to 90 degrees
- moved J1 33.1 mm to (194.1, 76.5), turned to 90 degrees
- moved U2 27.3 mm to (203.8, 45.1), turned to 270 degrees
- moved U4 17.2 mm to (190.2, 70.9), turned to 0 degrees
- moved J5 11.5 mm to (192.8, 44.0), turned to 270 degrees
- moved U5 4.35 mm to (197.0, 58.3)
- moved C2 3.91 mm to (211.5, 53.9)
- moved C1 3.68 mm to (215.2, 53.9), turned to 0 degrees
- moved J3 2.60 mm to (178.6, 58.2), turned to 0 degrees
- moved U3 1.90 mm to (197.3, 45.0)
- moved U1 1.80 mm to (213.2, 59.9)
Connections:
- U2 pad 8: CURRENT_FEEDBACK -> Net-(R1-Pad2)
- U5 pad 1: Net-(J3-Pad1) -> Net-(J3-Pad2)
- U5 pad 2: Net-(J3-Pad2) -> Net-(J3-Pad1)
Routing:
- net CURRENT_FEEDBACK: track 0.00 -> 43.2 mm, vias 0 -> 1
- net MOTOR_ENABLE: track 0.00 -> 35.7 mm
- net Net-(U2-Pad2): track 0.00 -> 34.2 mm
- net +12V: track 0.00 -> 27.2 mm, vias 0 -> 2
- net MODE: track 0.00 -> 21.7 mm, vias 0 -> 1
- net TX: track 0.00 -> 18.0 mm, vias 0 -> 1
- net MOTOR_STEP: track 0.00 -> 16.9 mm
- net RX: track 0.00 -> 14.8 mm, vias 0 -> 1
- net MOTOR_DIR: track 0.00 -> 10.2 mm
- net GND: track 0.00 -> 9.93 mm, vias 0 -> 6
- net Net-(J5-Pad2): track 0.00 -> 9.80 mm, vias 0 -> 1
- net Net-(J5-Pad4): track 0.00 -> 9.80 mm, vias 0 -> 1
- net Net-(J5-Pad3): track 0.00 -> 9.76 mm, vias 0 -> 1
- net Net-(J5-Pad1): track 0.00 -> 9.76 mm, vias 0 -> 1
- net RESET: track 0.00 -> 9.59 mm, vias 0 -> 1
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