File: Hardware/Electronics/CAD/MotorController.kicad_pcb (KiCad board)
At the start: 2 copper layers, 42.3 x 42.3 mm, 18 parts, among them J1 MPE 094-1-006, J2 CONN_01X03, J3 SolderTerminal, J5 CONN_01X04, SW2 SMD 4x4mm Button, U1 LD1117S33CTR, U2 MAX471, U3 TMC2130, U4 ESP-12E, U5 HiLink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

Commit message: new gerber files
Other:
- board text added: "Home Automation Stepper Motor Controller Revision 1.0.1 by Felix Kübler"
- board text removed: "Home Automation Stepper Motor Controller Layer Revision 1.0.0 by Felix Kübler"
Changed lines of the file:
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@@
     (links 58)
     (no_connects 1)
-    (area 175.883499 37.199499 218.324501 79.640501)
+    (area 171.541371 33.8819 220.807848 84.48099)
     (thickness 1.6)
-    (drawings 5)
+    (drawings 7)
     (tracks 187)
     (zones 0)
@@
       (drillshape 0)
       (scaleselection 1)
-      (outputdirectory gerber_data/))
+      (outputdirectory ../Gerber/))
   )
   (net 0 "")
@@
     )
   )
+  (dimension 42.418 (width 0.3) (layer Eco1.User)
+    (gr_text "42,418 mm" (at 196.977 33.448) (layer Eco1.User)
+      (effects (font (size 1.5 1.5) (thickness 0.3)))
+    )
+    (feature1 (pts (xy 218.186 37.084) (xy 218.186 32.098)))
+    (feature2 (pts (xy 175.768 37.084) (xy 175.768 32.098)))
+    (crossbar (pts (xy 175.768 34.798) (xy 218.186 34.798)))
+    (arrow1a (pts (xy 218.186 34.798) (xy 217.059496 35.384421)))
+    (arrow1b (pts (xy 218.186 34.798) (xy 217.059496 34.211579)))
+    (arrow2a (pts (xy 175.768 34.798) (xy 176.894504 35.384421)))
+    (arrow2b (pts (xy 175.768 34.798) (xy 176.894504 34.211579)))
+  )
+  (dimension 42.418 (width 0.3) (layer Eco1.User)
+    (gr_text "42,418 mm" (at 223.346 58.293 270) (layer Eco1.User)
+      (effects (font (size 1.5 1.5) (thickness 0.3)))
+    )
+    (feature1 (pts (xy 218.44 79.502) (xy 224.696 79.502)))
+    (feature2 (pts (xy 218.44 37.084) (xy 224.696 37.084)))
+    (crossbar (pts (xy 221.996 37.084) (xy 221.996 79.502)))
+    (arrow1a (pts (xy 221.996 79.502) (xy 221.409579 78.375496)))
+    (arrow1b (pts (xy 221.996 79.502) (xy 222.582421 78.375496)))
+    (arrow2a (pts (xy 221.996 37.084) (xy 221.409579 38.210504)))
+    (arrow2b (pts (xy 221.996 37.084) (xy 222.582421 38.210504)))
+  )
   (gr_line (start 218.2495 37.2745) (end 175.9585 37.2745) (angle 90) (layer Edge.Cuts) (width 0.15))
   (gr_line (start 218.2495 79.5655) (end 218.2495 37.2745) (angle 90) (layer Edge.Cuts) (width 0.15))
   (gr_line (start 175.9585 79.5655) (end 218.2495 79.5655) (angle 90) (layer Edge.Cuts) (width 0.15))
   (gr_line (start 175.9585 37.2745) (end 175.9585 79.5655) (angle 90) (layer Edge.Cuts) (width 0.15))
-  (gr_text "Home Automation\nStepper Motor Controller Layer\nRevision 1.0.0\nby Felix Kübler" (at 185.0644 71.12 270) (layer B.SilkS)
+  (gr_text "Home Automation\nStepper Motor Controller\nRevision 1.0.1\nby Felix Kübler" (at 185.0644 71.12 270) (layer B.SilkS)
     (effects (font (size 0.8 0.8) (thickness 0.125)) (justify left mirror))
   )
