File: Hardware/Electronics/CAD/MotorController.sch (KiCad schematic (older format))
At the start: 17 parts, among them J1 MPE 094-1-006, J2 CONN_01X03, J3 SolderTerminal, J5 CONN_01X04, SW2 Taster 9314, U1 LD1117S33CTR, U2 MAX471, U3 TMC2130, U4 ESP-12E, U5 HiLink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

Commit message: additional capacitor for current sensor smoothing
Parts:
- added C3: 0805 47uF, Capacitors_SMD:C_0805, symbol C
- C1, C2: value C -> 0805 10uF
- renumbered R5 to R4
Connections:
- net GND: now also C3.1
- net at R1.2, R3.2, U2.8 (OUT): now also C3.2
Other:
- moved on the sheet: R1, R2, R3
Changed lines of the file:
@@
 $EndComp
 $Comp
-L R R5
+L R R4
 U 1 1 599EC273
 P 3000 3350
-F 0 "R5" V 3080 3350 50  0000 C CNN
+F 0 "R4" V 3080 3350 50  0000 C CNN
 F 1 "RND 0805 1 10K" V 3150 3625 50  0000 C CNN
 F 2 "Resistors_SMD:R_0805" V 2930 3350 50  0001 C CNN
@@
 U 1 1 5A295074
 P 6025 3325
-F 0 "C2" H 6050 3425 50  0000 L CNN
-F 1 "C" H 6050 3225 50  0000 L CNN
+F 0 "C2" V 6175 3275 50  0000 L CNN
+F 1 "0805 10uF" V 6250 3150 50  0000 L CNN
 F 2 "Capacitors_SMD:C_0805" H 6063 3175 50  0001 C CNN
 F 3 "" H 6025 3325 50  0001 C CNN
@@
 U 1 1 5A295100
 P 5525 3325
-F 0 "C1" H 5550 3425 50  0000 L CNN
-F 1 "C" H 5550 3225 50  0000 L CNN
+F 0 "C1" V 5675 3275 50  0000 L CNN
+F 1 "0805 10uF" V 5750 3075 50  0000 L CNN
 F 2 "Capacitors_SMD:C_0805" H 5563 3175 50  0001 C CNN
 F 3 "" H 5525 3325 50  0001 C CNN
@@
 	0    -1   -1   0
 $EndComp
-Text GLabel 9150 2500 2    60   Input ~ 0
+Text GLabel 9775 2500 2    60   Input ~ 0
 CURRENT_FEEDBACK
 NoConn ~ 8375 2400
@@
 L R R1
 U 1 1 5ACA9F3E
-P 8750 2500
-F 0 "R1" V 8830 2500 50  0000 C CNN
-F 1 "RND 0805 1 100K" V 8900 2350 50  0000 C CNN
-F 2 "Resistors_SMD:R_0805" V 8680 2500 50  0001 C CNN
-F 3 "" H 8750 2500 50  0001 C CNN
-	1    8750 2500
+P 9375 2500
+F 0 "R1" V 9455 2500 50  0000 C CNN
+F 1 "RND 0805 1 100K" V 9525 2500 50  0000 C CNN
+F 2 "Resistors_SMD:R_0805" V 9305 2500 50  0001 C CNN
+F 3 "" H 9375 2500 50  0001 C CNN
+	1    9375 2500
 	0    1    1    0
 $EndComp
@@
 L R R2
 U 1 1 5ACAA259
-P 9300 2750
-F 0 "R2" V 9380 2750 50  0000 C CNN
-F 1 "RND 0805 1 47K" V 9450 3025 50  0000 C CNN
-F 2 "Resistors_SMD:R_0805" V 9230 2750 50  0001 C CNN
-F 3 "" H 9300 2750 50  0001 C CNN
-	1    9300 2750
-	0    1    1    0
-$EndComp
-Wire Wire Line
-	9000 2750 9150 2750
+P 9925 2750
+F 0 "R2" V 10005 2750 50  0000 C CNN
+F 1 "RND 0805 1 47K" V 10075 3025 50  0000 C CNN
+F 2 "Resistors_SMD:R_0805" V 9855 2750 50  0001 C CNN
+F 3 "" H 9925 2750 50  0001 C CNN
+	1    9925 2750
+	0    1    1    0
+$EndComp
+Wire Wire Line
+	9625 2750 9775 2750
 $Comp
 L GND #PWR22
 U 1 1 5ACAA303
-P 9550 2750
-F 0 "#PWR22" H 9550 2500 50  0001 C CNN
-F 1 "GND" V 9550 2550 50  0000 C CNN
-F 2 "" H 9550 2750 50  0001 C CNN
-F 3 "" H 9550 2750 50  0001 C CNN
-	1    9550 2750
-	0    -1   -1   0
-$EndComp
-Wire Wire Line
-	9450 2750 9550 2750
-Wire Wire Line
-	9000 2500 9000 2750
-Connection ~ 9000 2500
+P 10175 2750
+F 0 "#PWR22" H 10175 2500 50  0001 C CNN
+F 1 "GND" V 10175 2550 50  0000 C CNN
+F 2 "" H 10175 2750 50  0001 C CNN
+F 3 "" H 10175 2750 50  0001 C CNN
+	1    10175 2750
+	0    -1   -1   0
+$EndComp
+Wire Wire Line
+	10075 2750 10175 2750
+Wire Wire Line
+	9625 2500 9625 2750
+Connection ~ 9625 2500
 $Comp
 L R R3
 U 1 1 5B86C0A2
-P 8750 2300
-F 0 "R3" V 8575 2250 50  0000 C CNN
-F 1 "RND 0805 1 2K" V 8650 2550 50  0000 C CNN
-F 2 "Resistors_SMD:R_0805" V 8680 2300 50  0001 C CNN
-F 3 "" H 8750 2300 50  0001 C CNN
-	1    8750 2300
+P 9375 2300
+F 0 "R3" V 9200 2300 50  0000 C CNN
+F 1 "RND 0805 1 2K" V 9275 2300 50  0000 C CNN
+F 2 "Resistors_SMD:R_0805" V 9305 2300 50  0001 C CNN
+F 3 "" H 9375 2300 50  0001 C CNN
+	1    9375 2300
 	0    1    1    0
 $EndComp
@@
 L GND #PWR21
 U 1 1 5B86C312
-P 9000 2300
-F 0 "#PWR21" H 9000 2050 50  0001 C CNN
-F 1 "GND" V 8975 2100 50  0000 C CNN
-F 2 "" H 9000 2300 50  0001 C CNN
-F 3 "" H 9000 2300 50  0001 C CNN
-	1    9000 2300
-	0    -1   -1   0
-$EndComp
-Connection ~ 8500 2500
-Wire Wire Line
-	8375 2500 8600 2500
-Wire Wire Line
-	8500 2500 8500 2300
-Wire Wire Line
-	8900 2500 9150 2500
-Wire Wire Line
-	8500 2300 8600 2300
-Wire Wire Line
-	8900 2300 9000 2300
+P 9700 2100
+F 0 "#PWR21" H 9700 1850 50  0001 C CNN
+F 1 "GND" V 9675 1900 50  0000 C CNN
+F 2 "" H 9700 2100 50  0001 C CNN
+F 3 "" H 9700 2100 50  0001 C CNN
+	1    9700 2100
+	0    -1   -1   0
+$EndComp
+Connection ~ 9125 2500
+Wire Wire Line
+	8375 2500 9225 2500
+Wire Wire Line
+	9125 1950 9125 2500
+Wire Wire Line
+	9525 2500 9775 2500
+Wire Wire Line
+	9125 2300 9225 2300
+Wire Wire Line
+	9625 2300 9525 2300
+$Comp
+L C C3
+U 1 1 5B86CD6C
+P 9350 1950
+F 0 "C3" V 9150 1900 50  0000 L CNN
+F 1 "0805 47uF" V 9225 1775 50  0000 L CNN
+F 2 "Capacitors_SMD:C_0805" H 9388 1800 50  0001 C CNN
+F 3 "" H 9350 1950 50  0001 C CNN
+	1    9350 1950
+	0    1    1    0
+$EndComp
+Wire Wire Line
+	9125 1950 9200 1950
+Connection ~ 9125 2300
+Wire Wire Line
+	9700 2100 9625 2100
+Wire Wire Line
+	9625 1950 9625 2300
+Wire Wire Line
+	9625 1950 9500 1950
+Connection ~ 9625 2100
 $EndSCHEMATC

Commit message: library linkage fix
Parts:
- SW2: value Taster 9314 -> SMD 4x4mm Button
Connections:
- net RESET: now also SW2.2
Other:
- moved on the sheet: SW2
Changed lines of the file:
@@
 LIBS:Nema
 LIBS:TMC2130
+LIBS:SW_DPST_x2
 LIBS:MotorController-cache
 EELAYER 25 0
@@
 L SW_DPST_x2 SW2
 U 1 1 599EBC5A
-P 2450 3200
-F 0 "SW2" H 2450 3100 50  0000 C CNN
-F 1 "Taster 9314" H 2450 3025 50  0000 C CNN
-F 2 "Buttons_Switches_SMD:SW_SPST_SKQG" H 2450 3200 50  0001 C CNN
-F 3 "" H 2450 3200 50  0001 C CNN
-	1    2450 3200
+P 2300 3200
+F 0 "SW2" H 2300 3100 50  0000 C CNN
+F 1 "SMD 4x4mm Button" H 2300 3025 50  0000 C CNN
+F 2 "Buttons_Switches_SMD:SW_SPST_SKQG" H 2300 3200 50  0001 C CNN
+F 3 "" H 2300 3200 50  0001 C CNN
+	1    2300 3200
 	1    0    0    -1
 $EndComp
@@
 L +3.3V #PWR1
 U 1 1 599EBD49
-P 2100 3200
-F 0 "#PWR1" H 2100 3050 50  0001 C CNN
-F 1 "+3.3V" V 2100 3450 50  0000 C CNN
-F 2 "" H 2100 3200 50  0001 C CNN
-F 3 "" H 2100 3200 50  0001 C CNN
-	1    2100 3200
+P 1800 3200
+F 0 "#PWR1" H 1800 3050 50  0001 C CNN
+F 1 "+3.3V" V 1800 3450 50  0000 C CNN
+F 2 "" H 1800 3200 50  0001 C CNN
+F 3 "" H 1800 3200 50  0001 C CNN
+	1    1800 3200
 	0    -1   -1   0
 $EndComp
@@
 	4750 6400 5300 6400
 Wire Wire Line
-	2100 3200 2250 3200
+	1800 3200 1950 3200
 Wire Wire Line
 	3150 3350 3300 3350

Commit message: terminal footprints
Parts:
- J3: footprint Terminal:SolderTerminal -> Terminal:SolderPad_1x2_2.54mm
- J5: footprint Terminal:Pin_Header_SMD_Angled_2.54mm -> Terminal:Pin_Header_SMD_1x4_Angled_2.54mm
Changed lines of the file:
@@
 LIBS:TMC2130
 LIBS:SW_DPST_x2
-LIBS:MotorController-cache
 EELAYER 25 0
 EELAYER END
@@
 $EndComp
 $Comp
-L GND #PWR9
+L GND #PWR01
 U 1 1 592C2849
 P 4950 6600
-F 0 "#PWR9" H 4950 6350 50  0001 C CNN
+F 0 "#PWR01" H 4950 6350 50  0001 C CNN
 F 1 "GND" V 4850 6525 50  0000 C CNN
 F 2 "" H 4950 6600 50  0001 C CNN
@@
 $EndComp
 $Comp
-L +3.3V #PWR3
+L +3.3V #PWR02
 U 1 1 592C2C75
 P 2750 6600
-F 0 "#PWR3" H 2750 6450 50  0001 C CNN
+F 0 "#PWR02" H 2750 6450 50  0001 C CNN
 F 1 "+3.3V" V 2650 6675 50  0000 C CNN
 F 2 "" H 2750 6600 50  0001 C CNN
@@
 $EndComp
 $Comp
-L +3.3V #PWR2
+L +3.3V #PWR03
 U 1 1 592C2CAB
 P 2750 6100
-F 0 "#PWR2" H 2750 5950 50  0001 C CNN
+F 0 "#PWR03" H 2750 5950 50  0001 C CNN
 F 1 "+3.3V" V 2750 6350 50  0000 C CNN
 F 2 "" H 2750 6100 50  0001 C CNN
@@
 NoConn ~ 3900 7100
 $Comp
-L GND #PWR5
+L GND #PWR04
 U 1 1 592C460C
 P 2850 1775
-F 0 "#PWR5" H 2850 1525 50  0001 C CNN
+F 0 "#PWR04" H 2850 1525 50  0001 C CNN
 F 1 "GND" V 2900 1575 50  0000 C CNN
 F 2 "" H 2850 1775 50  0001 C CNN
@@
 MODE
 $Comp
-L GND #PWR6
+L GND #PWR05
 U 1 1 592C5F8F
 P 2900 2425
-F 0 "#PWR6" H 2900 2175 50  0001 C CNN
+F 0 "#PWR05" H 2900 2175 50  0001 C CNN
 F 1 "GND" V 2900 2225 50  0000 C CNN
 F 2 "" H 2900 2425 50  0001 C CNN
@@
 $EndComp
 $Comp
-L +3.3V #PWR7
+L +3.3V #PWR06
 U 1 1 592C600F
 P 2900 2625
-F 0 "#PWR7" H 2900 2475 50  0001 C CNN
+F 0 "#PWR06" H 2900 2475 50  0001 C CNN
 F 1 "+3.3V" V 2900 2875 50  0000 C CNN
 F 2 "" H 2900 2625 50  0001 C CNN
@@
 $EndComp
 $Comp
-L +3.3V #PWR11
+L +3.3V #PWR07
 U 1 1 595EB4E9
 P 5300 6400
-F 0 "#PWR11" H 5300 6250 50  0001 C CNN
+F 0 "#PWR07" H 5300 6250 50  0001 C CNN
 F 1 "+3.3V" V 5350 6600 50  0000 C CNN
 F 2 "" H 5300 6400 50  0001 C CNN
@@
 $EndComp
 $Comp
-L +3.3V #PWR1
+L +3.3V #PWR08
 U 1 1 599EBD49
 P 1800 3200
-F 0 "#PWR1" H 1800 3050 50  0001 C CNN
+F 0 "#PWR08" H 1800 3050 50  0001 C CNN
 F 1 "+3.3V" V 1800 3450 50  0000 C CNN
 F 2 "" H 1800 3200 50  0001 C CNN
@@
 $EndComp
 $Comp
-L GND #PWR8
+L GND #PWR09
 U 1 1 599EC69C
 P 3300 3350
-F 0 "#PWR8" H 3300 3100 50  0001 C CNN
+F 0 "#PWR09" H 3300 3100 50  0001 C CNN
 F 1 "GND" V 3300 3150 50  0000 C CNN
 F 2 "" H 3300 3350 50  0001 C CNN
@@
 RESET
 $Comp
-L +3.3V #PWR4
+L +3.3V #PWR010
 U 1 1 5A1C2463
 P 2850 1575
-F 0 "#PWR4" H 2850 1425 50  0001 C CNN
+F 0 "#PWR010" H 2850 1425 50  0001 C CNN
 F 1 "+3.3V" V 2775 1800 50  0000 C CNN
 F 2 "" H 2850 1575 50  0001 C CNN
@@
 $EndComp
 $Comp
-L +3.3V #PWR13
+L +3.3V #PWR011
 U 1 1 5A294EEF
 P 6325 2975
-F 0 "#PWR13" H 6325 2825 50  0001 C CNN
+F 0 "#PWR011" H 6325 2825 50  0001 C CNN
 F 1 "+3.3V" V 6325 3200 50  0000 C CNN
 F 2 "" H 6325 2975 50  0001 C CNN
@@
 $EndComp
 $Comp
-L +12V #PWR10
+L +12V #PWR012
 U 1 1 5A294F1E
 P 5225 2975
-F 0 "#PWR10" H 5225 2825 50  0001 C CNN
+F 0 "#PWR012" H 5225 2825 50  0001 C CNN
 F 1 "+12V" V 5225 3200 50  0000 C CNN
 F 2 "" H 5225 2975 50  0001 C CNN
@@
 $EndComp
 $Comp
-L GND #PWR12
+L GND #PWR013
 U 1 1 5A294F4D
 P 5775 3425
-F 0 "#PWR12" H 5775 3175 50  0001 C CNN
+F 0 "#PWR013" H 5775 3175 50  0001 C CNN
 F 1 "GND" V 5775 3225 50  0000 C CNN
 F 2 "" H 5775 3425 50  0001 C CNN
@@
 MOTOR_STEP
 $Comp
-L +3.3V #PWR15
+L +3.3V #PWR014
 U 1 1 5A2EB86A
 P 6900 4425
-F 0 "#PWR15" H 6900 4275 50  0001 C CNN
+F 0 "#PWR014" H 6900 4275 50  0001 C CNN
 F 1 "+3.3V" V 6900 4675 50  0000 C CNN
 F 2 "" H 6900 4425 50  0001 C CNN
@@
 $EndComp
 $Comp
-L GND #PWR14
+L GND #PWR015
 U 1 1 5A2EB8A2
 P 6900 4325
-F 0 "#PWR14" H 6900 4075 50  0001 C CNN
+F 0 "#PWR015" H 6900 4075 50  0001 C CNN
 F 1 "GND" V 6900 4100 50  0000 C CNN
 F 2 "" H 6900 4325 50  0001 C CNN
@@
 F 0 "J5" H 6350 5025 50  0000 C CNN
 F 1 "CONN_01X04" H 6525 4925 50  0000 C CNN
-F 2 "Terminal:Pin_Header_SMD_Angled_2.54mm" H 6350 4675 50  0001 C CNN
+F 2 "Terminal:Pin_Header_SMD_1x4_Angled_2.54mm" H 6350 4675 50  0001 C CNN
 F 3 "" H 6350 4675 50  0001 C CNN
 	1    6350 4675
@@
 $EndComp
 $Comp
-L GND #PWR16
+L GND #PWR016
 U 1 1 5A2EC268
 P 6900 4925
-F 0 "#PWR16" H 6900 4675 50  0001 C CNN
+F 0 "#PWR016" H 6900 4675 50  0001 C CNN
 F 1 "GND" V 6900 4700 50  0000 C CNN
 F 2 "" H 6900 4925 50  0001 C CNN
@@
 $EndComp
 $Comp
-L +12V #PWR17
+L +12V #PWR017
 U 1 1 5A2EC2F3
 P 6900 5025
-F 0 "#PWR17" H 6900 4875 50  0001 C CNN
+F 0 "#PWR017" H 6900 4875 50  0001 C CNN
 F 1 "+12V" V 6900 5250 50  0000 C CNN
 F 2 "" H 6900 5025 50  0001 C CNN
@@
 F 0 "J3" H 5975 1725 50  0000 C TNN
 F 1 "SolderTerminal" H 5750 1800 50  0000 C TNN
-F 2 "Terminal:SolderTerminal" H 5925 1775 50  0001 C CNN
+F 2 "Terminal:SolderPad_1x2_2.54mm" H 5925 1775 50  0001 C CNN
 F 3 "" H 5900 2000 50  0001 C CNN
 	1    5925 2000
@@
 $EndComp
 $Comp
-L +12V #PWR20
+L +12V #PWR018
 U 1 1 5AC69F04
 P 8475 2100
-F 0 "#PWR20" H 8475 1950 50  0001 C CNN
+F 0 "#PWR018" H 8475 1950 50  0001 C CNN
 F 1 "+12V" V 8375 2225 50  0000 C CNN
 F 2 "" H 8475 2100 50  0001 C CNN
@@
 $EndComp
 $Comp
-L GND #PWR18
+L GND #PWR019
 U 1 1 5AC69F36
 P 7125 1900
-F 0 "#PWR18" H 7125 1650 50  0001 C CNN
+F 0 "#PWR019" H 7125 1650 50  0001 C CNN
 F 1 "GND" V 7125 1700 50  0000 C CNN
 F 2 "" H 7125 1900 50  0001 C CNN
@@
 NoConn ~ 8375 2400
 $Comp
-L GND #PWR19
+L GND #PWR020
 U 1 1 5AC6B0DF
 P 7475 2500
-F 0 "#PWR19" H 7475 2250 50  0001 C CNN
+F 0 "#PWR020" H 7475 2250 50  0001 C CNN
 F 1 "GND" V 7475 2300 50  0000 C CNN
 F 2 "" H 7475 2500 50  0001 C CNN
@@
 	9625 2750 9775 2750
 $Comp
-L GND #PWR22
+L GND #PWR021
 U 1 1 5ACAA303
 P 10175 2750
-F 0 "#PWR22" H 10175 2500 50  0001 C CNN
+F 0 "#PWR021" H 10175 2500 50  0001 C CNN
 F 1 "GND" V 10175 2550 50  0000 C CNN
 F 2 "" H 10175 2750 50  0001 C CNN
@@
 $EndComp
 $Comp
-L GND #PWR21
+L GND #PWR022
 U 1 1 5B86C312
 P 9700 2100
-F 0 "#PWR21" H 9700 1850 50  0001 C CNN
+F 0 "#PWR022" H 9700 1850 50  0001 C CNN
 F 1 "GND" V 9675 1900 50  0000 C CNN
 F 2 "" H 9700 2100 50  0001 C CNN
